Commit message: fix the package names

File: rebel_arm_description/urdf/arm.xacro (robot description, xacro)
@@ -1,7 +1,7 @@
 <?xml version="1.0" ?>
 <robot name="arm" xmlns:xacro="http://www.ros.org/wiki/xacro">
-<xacro:include filename="$(find arm_description)/urdf/materials.xacro" />
-<xacro:include filename="$(find arm_description)/urdf/arm.trans" />
-<xacro:include filename="$(find arm_description)/urdf/arm.gazebo" />
+<xacro:include filename="$(find rebel_arm_description)/urdf/materials.xacro" />
+<xacro:include filename="$(find rebel_arm_description)/urdf/arm.trans" />
+<xacro:include filename="$(find rebel_arm_description)/urdf/arm.gazebo" />
 <link name="base_link">
   <inertial>
@@ -13,5 +13,5 @@
     <origin xyz="0 0 0" rpy="0 0 0"/>
     <geometry>
-      <mesh filename="file://$(find arm_description)/meshes/base_link.stl" scale="0.001 0.001 0.001"/>
+      <mesh filename="file://$(find rebel_arm_description)/meshes/base_link.stl" scale="0.001 0.001 0.001"/>
     </geometry>
     <material name="silver"/>
@@ -20,5 +20,5 @@
     <origin xyz="0 0 0" rpy="0 0 0"/>
     <geometry>
-      <mesh filename="file://$(find arm_description)/meshes/base_link.stl" scale="0.001 0.001 0.001"/>
+      <mesh filename="file://$(find rebel_arm_description)/meshes/base_link.stl" scale="0.001 0.001 0.001"/>
     </geometry>
   </collision>
@@ -33,5 +33,5 @@
     <origin xyz="-0.0 -0.0 -0.09" rpy="0 0 0"/>
     <geometry>
-      <mesh filename="file://$(find arm_description)/meshes/pulley_c_v9_1.stl" scale="0.001 0.001 0.001"/>
+      <mesh filename="file://$(find rebel_arm_description)/meshes/pulley_c_v9_1.stl" scale="0.001 0.001 0.001"/>
     </geometry>
     <material name="silver"/>
@@ -40,5 +40,5 @@
     <origin xyz="-0.0 -0.0 -0.09" rpy="0 0 0"/>
     <geometry>
-      <mesh filename="file://$(find arm_description)/meshes/pulley_c_v9_1.stl" scale="0.001 0.001 0.001"/>
+      <mesh filename="file://$(find rebel_arm_description)/meshes/pulley_c_v9_1.stl" scale="0.001 0.001 0.001"/>
     </geometry>
   </collision>
@@ -53,5 +53,5 @@
     <origin xyz="-0.0 -0.0 -0.123" rpy="0 0 0"/>
     <geometry>
-      <mesh filename="file://$(find arm_description)/meshes/shoulder_bearling_house_prt1_v14_1.stl" scale="0.001 0.001 0.001"/>
+      <mesh filename="file://$(find rebel_arm_description)/meshes/shoulder_bearling_house_prt1_v14_1.stl" scale="0.001 0.001 0.001"/>
     </geometry>
     <material name="silver"/>
@@ -60,5 +60,5 @@
     <origin xyz="-0.0 -0.0 -0.123" rpy="0 0 0"/>
     <geometry>
-      <mesh filename="file://$(find arm_description)/meshes/shoulder_bearling_house_prt1_v14_1.stl" scale="0.001 0.001 0.001"/>
+      <mesh filename="file://$(find rebel_arm_description)/meshes/shoulder_bearling_house_prt1_v14_1.stl" scale="0.001 0.001 0.001"/>
     </geometry>
   </collision>
@@ -73,5 +73,5 @@
     <origin xyz="-0.0 -0.0 -0.1344" rpy="0 0 0"/>
     <geometry>
-      <mesh filename="file://$(find arm_description)/meshes/table1_v2_1.stl" scale="0.001 0.001 0.001"/>
+      <mesh filename="file://$(find rebel_arm_description)/meshes/table1_v2_1.stl" scale="0.001 0.001 0.001"/>
     </geometry>
     <material name="silver"/>
@@ -80,5 +80,5 @@
     <origin xyz="-0.0 -0.0 -0.1344" rpy="0 0 0"/>
     <geometry>
-      <mesh filename="file://$(find arm_description)/meshes/table1_v2_1.stl" scale="0.001 0.001 0.001"/>
+      <mesh filename="file://$(find rebel_arm_description)/meshes/table1_v2_1.stl" scale="0.001 0.001 0.001"/>
     </geometry>
   </collision>
@@ -93,5 +93,5 @@
     <origin xyz="-0.0 -0.0 -0.1504" rpy="0 0 0"/>
     <geometry>
-      <mesh filename="file://$(find arm_description)/meshes/shoulder_bearling_house_prt3_v2_1.stl" scale="0.001 0.001 0.001"/>
+      <mesh filename="file://$(find rebel_arm_description)/meshes/shoulder_bearling_house_prt3_v2_1.stl" scale="0.001 0.001 0.001"/>
     </geometry>
     <material name="silver"/>
@@ -100,5 +100,5 @@
     <origin xyz="-0.0 -0.0 -0.1504" rpy="0 0 0"/>
     <geometry>
-      <mesh filename="file://$(find arm_description)/meshes/shoulder_bearling_house_prt3_v2_1.stl" scale="0.001 0.001 0.001"/>
+      <mesh filename="file://$(find rebel_arm_description)/meshes/shoulder_bearling_house_prt3_v2_1.stl" scale="0.001 0.001 0.001"/>
     </geometry>
   </collision>
@@ -113,5 +113,5 @@
     <origin xyz="-0.05 0.095 -0.1504" rpy="0 0 0"/>
     <geometry>
-      <mesh filename="file://$(find arm_description)/meshes/shoulder_v2_1.stl" scale="0.001 0.001 0.001"/>
+      <mesh filename="file://$(find rebel_arm_description)/meshes/shoulder_v2_1.stl" scale="0.001 0.001 0.001"/>
     </geometry>
     <material name="silver"/>
@@ -120,5 +120,5 @@
     <origin xyz="-0.05 0.095 -0.1504" rpy="0 0 0"/>
     <geometry>
-      <mesh filename="file://$(find arm_description)/meshes/shoulder_v2_1.stl" scale="0.001 0.001 0.001"/>
+      <mesh filename="file://$(find rebel_arm_description)/meshes/shoulder_v2_1.stl" scale="0.001 0.001 0.001"/>
     </geometry>
   </collision>
@@ -133,5 +133,5 @@
     <origin xyz="2.4e-05 0.097184 -0.1954" rpy="0 0 0"/>
     <geometry>
-      <mesh filename="file://$(find arm_description)/meshes/plangearbox1_v2_1.stl" scale="0.001 0.001 0.001"/>
+      <mesh filename="file://$(find rebel_arm_description)/meshes/plangearbox1_v2_1.stl" scale="0.001 0.001 0.001"/>
     </geometry>
     <material name="silver"/>
@@ -140,5 +140,5 @@
     <origin xyz="2.4e-05 0.097184 -0.1954" rpy="0 0 0"/>
     <geometry>
-      <mesh filename="file://$(find arm_description)/meshes/plangearbox1_v2_1.stl" scale="0.001 0.001 0.001"/>
+      <mesh filename="file://$(find rebel_arm_description)/meshes/plangearbox1_v2_1.stl" scale="0.001 0.001 0.001"/>
     </geometry>
   </collision>
@@ -153,5 +153,5 @@
     <origin xyz="6.7e-05 0.013684 -0.1954" rpy="0 0 0"/>
     <geometry>
-      <mesh filename="file://$(find arm_description)/meshes/stepper1_v2_1.stl" scale="0.001 0.001 0.001"/>
+      <mesh filename="file://$(find rebel_arm_description)/meshes/stepper1_v2_1.stl" scale="0.001 0.001 0.001"/>
     </geometry>
     <material name="silver"/>
@@ -160,5 +160,5 @@
     <origin xyz="6.7e-05 0.013684 -0.1954" rpy="0 0 0"/>
     <geometry>
-      <mesh filename="file://$(find arm_description)/meshes/stepper1_v2_1.stl" scale="0.001 0.001 0.001"/>
+      <mesh filename="file://$(find rebel_arm_description)/meshes/stepper1_v2_1.stl" scale="0.001 0.001 0.001"/>
     </geometry>
   </collision>
@@ -173,5 +173,5 @@
     <origin xyz="4.5e-05 0.055884 -0.2754" rpy="0 0 0"/>
     <geometry>
-      <mesh filename="file://$(find arm_description)/meshes/shoulder_bearling_house2_prt3_v3_1.stl" scale="0.001 0.001 0.001"/>
+      <mesh filename="file://$(find rebel_arm_description)/meshes/shoulder_bearling_house2_prt3_v3_1.stl" scale="0.001 0.001 0.001"/>
     </geometry>
     <material name="silver"/>
@@ -180,5 +180,5 @@
     <origin xyz="4.5e-05 0.055884 -0.2754" rpy="0 0 0"/>
     <geometry>
-      <mesh filename="file://$(find arm_description)/meshes/shoulder_bearling_house2_prt3_v3_1.stl" scale="0.001 0.001 0.001"/>
+      <mesh filename="file://$(find rebel_arm_description)/meshes/shoulder_bearling_house2_prt3_v3_1.stl" scale="0.001 0.001 0.001"/>
     </geometry>
   </collision>
@@ -193,5 +193,5 @@
     <origin xyz="2.1e-05 0.102029 -0.2754" rpy="0 0 0"/>
     <geometry>
-      <mesh filename="file://$(find arm_description)/meshes/new_pipe_b_v8_1.stl" scale="0.001 0.001 0.001"/>
+      <mesh filename="file://$(find rebel_arm_description)/meshes/new_pipe_b_v8_1.stl" scale="0.001 0.001 0.001"/>
     </geometry>
     <material name="silver"/>
@@ -200,5 +200,5 @@
     <origin xyz="2.1e-05 0.102029 -0.2754" rpy="0 0 0"/>
     <geometry>
-      <mesh filename="file://$(find arm_description)/meshes/new_pipe_b_v8_1.stl" scale="0.001 0.001 0.001"/>
+      <mesh filename="file://$(find rebel_arm_description)/meshes/new_pipe_b_v8_1.stl" scale="0.001 0.001 0.001"/>
     </geometry>
   </collision>
@@ -213,5 +213,5 @@
     <origin xyz="2.1e-05 0.102029 -0.2754" rpy="0 0 0"/>
     <geometry>
-      <mesh filename="file://$(find arm_description)/meshes/shoulder_bearling_house_2prt1_v5_1.stl" scale="0.001 0.001 0.001"/>
+      <mesh filename="file://$(find rebel_arm_description)/meshes/shoulder_bearling_house_2prt1_v5_1.stl" scale="0.001 0.001 0.001"/>
     </geometry>
     <material name="silver"/>
@@ -220,5 +220,5 @@
     <origin xyz="2.1e-05 0.102029 -0.2754" rpy="0 0 0"/>
     <geometry>
-      <mesh filename="file://$(find arm_description)/meshes/shoulder_bearling_house_2prt1_v5_1.stl" scale="0.001 0.001 0.001"/>
+      <mesh filename="file://$(find rebel_arm_description)/meshes/shoulder_bearling_house_2prt1_v5_1.stl" scale="0.001 0.001 0.001"/>
     </geometry>
   </collision>
@@ -233,5 +233,5 @@
     <origin xyz="3e-05 0.085884 -0.2754" rpy="0 0 0"/>
     <geometry>
-      <mesh filename="file://$(find arm_description)/meshes/shoulder_bearling_house2_prt2_v10_1.stl" scale="0.001 0.001 0.001"/>
+      <mesh filename="file://$(find rebel_arm_description)/meshes/shoulder_bearling_house2_prt2_v10_1.stl" scale="0.001 0.001 0.001"/>
     </geometry>
     <material name="silver"/>
@@ -240,5 +240,5 @@
     <origin xyz="3e-05 0.085884 -0.2754" rpy="0 0 0"/>
     <geometry>
-      <mesh filename="file://$(find arm_description)/meshes/shoulder_bearling_house2_prt2_v10_1.stl" scale="0.001 0.001 0.001"/>
+      <mesh filename="file://$(find rebel_arm_description)/meshes/shoulder_bearling_house2_prt2_v10_1.stl" scale="0.001 0.001 0.001"/>
     </geometry>
   </collision>
@@ -253,5 +253,5 @@
     <origin xyz="9.6e-05 -0.042971 -0.2754" rpy="0 0 0"/>
     <geometry>
-      <mesh filename="file://$(find arm_description)/meshes/tbone_v1_1.stl" scale="0.001 0.001 0.001"/>
+      <mesh filename="file://$(find rebel_arm_description)/meshes/tbone_v1_1.stl" scale="0.001 0.001 0.001"/>
     </geometry>
     <material name="silver"/>
@@ -260,5 +260,5 @@
     <origin xyz="9.6e-05 -0.042971 -0.2754" rpy="0 0 0"/>
     <geometry>
-      <mesh filename="file://$(find arm_description)/meshes/tbone_v1_1.stl" scale="0.001 0.001 0.001"/>
+      <mesh filename="file://$(find rebel_arm_description)/meshes/tbone_v1_1.stl" scale="0.001 0.001 0.001"/>
     </geometry>
   </collision>
@@ -273,5 +273,5 @@
     <origin xyz="0.0002 -0.002971 -0.308202" rpy="0 0 0"/>
     <geometry>
-      <mesh filename="file://$(find arm_description)/meshes/pipe_c_v1_1.stl" scale="0.001 0.001 0.001"/>
+      <mesh filename="file://$(find rebel_arm_description)/meshes/pipe_c_v1_1.stl" scale="0.001 0.001 0.001"/>
     </geometry>
     <material name="silver"/>
@@ -280,5 +280,5 @@
     <origin xyz="0.0002 -0.002971 -0.308202" rpy="0 0 0"/>
     <geometry>
-      <mesh filename="file://$(find arm_description)/meshes/pipe_c_v1_1.stl" scale="0.001 0.001 0.001"/>
+      <mesh filename="file://$(find rebel_arm_description)/meshes/pipe_c_v1_1.stl" scale="0.001 0.001 0.001"/>
     </geometry>
   </collision>
@@ -293,5 +293,5 @@
     <origin xyz="0.0002 -0.002971 -0.368202" rpy="0 0 0"/>
     <geometry>
-      <mesh filename="file://$(find arm_description)/meshes/table2_v1_1.stl" scale="0.001 0.001 0.001"/>
+      <mesh filename="file://$(find rebel_arm_description)/meshes/table2_v1_1.stl" scale="0.001 0.001 0.001"/>
     </geometry>
     <material name="silver"/>
@@ -300,5 +300,5 @@
     <origin xyz="0.0002 -0.002971 -0.368202" rpy="0 0 0"/>
     <geometry>
-      <mesh filename="file://$(find arm_description)/meshes/table2_v1_1.stl" scale="0.001 0.001 0.001"/>
+      <mesh filename="file://$(find rebel_arm_description)/meshes/table2_v1_1.stl" scale="0.001 0.001 0.001"/>
     </geometry>
   </collision>
@@ -313,5 +313,5 @@
     <origin xyz="0.000157 0.081029 -0.398202" rpy="0 0 0"/>
     <geometry>
-      <mesh filename="file://$(find arm_description)/meshes/arm_plate_v2_1.stl" scale="0.001 0.001 0.001"/>
+      <mesh filename="file://$(find rebel_arm_description)/meshes/arm_plate_v2_1.stl" scale="0.001 0.001 0.001"/>
     </geometry>
     <material name="silver"/>
@@ -320,5 +320,5 @@
     <origin xyz="0.000157 0.081029 -0.398202" rpy="0 0 0"/>
     <geometry>
-      <mesh filename="file://$(find arm_description)/meshes/arm_plate_v2_1.stl" scale="0.001 0.001 0.001"/>
+      <mesh filename="file://$(find rebel_arm_description)/meshes/arm_plate_v2_1.stl" scale="0.001 0.001 0.001"/>
     </geometry>
   </collision>
@@ -333,5 +333,5 @@
     <origin xyz="0.000156 0.082029 -0.628362" rpy="0 0 0"/>
     <geometry>
-      <mesh filename="file://$(find arm_description)/meshes/bearing_holder_elbow_v3_1.stl" scale="0.001 0.001 0.001"/>
+      <mesh filename="file://$(find rebel_arm_description)/meshes/bearing_holder_elbow_v3_1.stl" scale="0.001 0.001 0.001"/>
     </geometry>
     <material name="silver"/>
@@ -340,5 +340,5 @@
     <origin xyz="0.000156 0.082029 -0.628362" rpy="0 0 0"/>
     <geometry>
-      <mesh filename="file://$(find arm_description)/meshes/bearing_holder_elbow_v3_1.stl" scale="0.001 0.001 0.001"/>
+      <mesh filename="file://$(find rebel_arm_description)/meshes/bearing_holder_elbow_v3_1.stl" scale="0.001 0.001 0.001"/>
     </geometry>
   </collision>
@@ -353,5 +353,5 @@
     <origin xyz="0.000151 0.091029 -0.628362" rpy="0 0 0"/>
     <geometry>
-      <mesh filename="file://$(find arm_description)/meshes/elbow_joint_axes_v5_1.stl" scale="0.001 0.001 0.001"/>
+      <mesh filename="file://$(find rebel_arm_description)/meshes/elbow_joint_axes_v5_1.stl" scale="0.001 0.001 0.001"/>
     </geometry>
     <material name="silver"/>
@@ -360,5 +360,5 @@
     <origin xyz="0.000151 0.091029 -0.628362" rpy="0 0 0"/>
     <geometry>
-      <mesh filename="file://$(find arm_description)/meshes/elbow_joint_axes_v5_1.stl" scale="0.001 0.001 0.001"/>
+      <mesh filename="file://$(find rebel_arm_description)/meshes/elbow_joint_axes_v5_1.stl" scale="0.001 0.001 0.001"/>
     </geometry>
   </collision>
@@ -373,5 +373,5 @@
     <origin xyz="0.000174 0.047929 -0.628362" rpy="0 0 0"/>
     <geometry>
-      <mesh filename="file://$(find arm_description)/meshes/elbow_side_plate_v3_1.stl" scale="0.001 0.001 0.001"/>
+      <mesh filename="file://$(find rebel_arm_description)/meshes/elbow_side_plate_v3_1.stl" scale="0.001 0.001 0.001"/>
     </geometry>
     <material name="silver"/>
@@ -380,5 +380,5 @@
     <origin xyz="0.000174 0.047929 -0.628362" rpy="0 0 0"/>
     <geometry>
-      <mesh filename="file://$(find arm_description)/meshes/elbow_side_plate_v3_1.stl" scale="0.001 0.001 0.001"/>
+      <mesh filename="file://$(find rebel_arm_description)/meshes/elbow_side_plate_v3_1.stl" scale="0.001 0.001 0.001"/>
     </geometry>
   </collision>
@@ -393,5 +393,5 @@
     <origin xyz="-0.075429 0.052391 -0.628362" rpy="0 0 0"/>
     <geometry>
-      <mesh filename="file://$(find arm_description)/meshes/elbow_pipe_holder_front_v1_1.stl" scale="0.001 0.001 0.001"/>
+      <mesh filename="file://$(find rebel_arm_description)/meshes/elbow_pipe_holder_front_v1_1.stl" scale="0.001 0.001 0.001"/>
     </geometry>
     <material name="silver"/>
@@ -400,5 +400,5 @@
     <origin xyz="-0.075429 0.052391 -0.628362" rpy="0 0 0"/>
     <geometry>
-      <mesh filename="file://$(find arm_description)/meshes/elbow_pipe_holder_front_v1_1.stl" scale="0.001 0.001 0.001"/>
+      <mesh filename="file://$(find rebel_arm_description)/meshes/elbow_pipe_holder_front_v1_1.stl" scale="0.001 0.001 0.001"/>
     </geometry>
   </collision>
@@ -413,5 +413,5 @@
     <origin xyz="0.044573 0.050002 -0.628362" rpy="0 0 0"/>
     <geometry>
-      <mesh filename="file://$(find arm_description)/meshes/elbow_pipe_holder_rear_v1_1.stl" scale="0.001 0.001 0.001"/>
+      <mesh filename="file://$(find rebel_arm_description)/meshes/elbow_pipe_holder_rear_v1_1.stl" scale="0.001 0.001 0.001"/>
     </geometry>
     <material name="silver"/>
@@ -420,5 +420,5 @@
     <origin xyz="0.044573 0.050002 -0.628362" rpy="0 0 0"/>
     <geometry>
-      <mesh filename="file://$(find arm_description)/meshes/elbow_pipe_holder_rear_v1_1.stl" scale="0.001 0.001 0.001"/>
+      <mesh filename="file://$(find rebel_arm_description)/meshes/elbow_pipe_holder_rear_v1_1.stl" scale="0.001 0.001 0.001"/>
     </geometry>
   </collision>
@@ -433,5 +433,5 @@
     <origin xyz="0.038602 -0.006274 -0.628362" rpy="0 0 0"/>
     <geometry>
-      <mesh filename="file://$(find arm_description)/meshes/pipe_under_arm_v2_1.stl" scale="0.001 0.001 0.001"/>
+      <mesh filename="file://$(find rebel_arm_description)/meshes/pipe_under_arm_v2_1.stl" scale="0.001 0.001 0.001"/>
     </geometry>
     <material name="silver"/>
@@ -440,5 +440,5 @@
     <origin xyz="0.038602 -0.006274 -0.628362" rpy="0 0 0"/>
     <geometry>
-      <mesh filename="file://$(find arm_description)/meshes/pipe_under_arm_v2_1.stl" scale="0.001 0.001 0.001"/>
+      <mesh filename="file://$(find rebel_arm_description)/meshes/pipe_under_arm_v2_1.stl" scale="0.001 0.001 0.001"/>
     </geometry>
   </collision>
@@ -453,5 +453,5 @@
     <origin xyz="-0.181398 -0.006388 -0.628362" rpy="0 0 0"/>
     <geometry>
-      <mesh filename="file://$(find arm_description)/meshes/hand_joint_mount_plate_v3_1.stl" scale="0.001 0.001 0.001"/>
+      <mesh filename="file://$(find rebel_arm_description)/meshes/hand_joint_mount_plate_v3_1.stl" scale="0.001 0.001 0.001"/>
     </geometry>
     <material name="silver"/>
@@ -460,5 +460,5 @@
     <origin xyz="-0.181398 -0.006388 -0.628362" rpy="0 0 0"/>
     <geometry>
-      <mesh filename="file://$(find arm_description)/meshes/hand_joint_mount_plate_v3_1.stl" scale="0.001 0.001 0.001"/>
+      <mesh filename="file://$(find rebel_arm_description)/meshes/hand_joint_mount_plate_v3_1.stl" scale="0.001 0.001 0.001"/>
     </geometry>
   </collision>
@@ -473,5 +473,5 @@
     <origin xyz="-0.187433 0.060609 -0.659562" rpy="0 0 0"/>
     <geometry>
-      <mesh filename="file://$(find arm_description)/meshes/hand_joint_side_plate_v4_1.stl" scale="0.001 0.001 0.001"/>
+      <mesh filename="file://$(find rebel_arm_description)/meshes/hand_joint_side_plate_v4_1.stl" scale="0.001 0.001 0.001"/>
     </geometry>
     <material name="silver"/>
@@ -480,5 +480,5 @@
     <origin xyz="-0.187433 0.060609 -0.659562" rpy="0 0 0"/>
     <geometry>
-      <mesh filename="file://$(find arm_description)/meshes/hand_joint_side_plate_v4_1.stl" scale="0.001 0.001 0.001"/>
+      <mesh filename="file://$(find rebel_arm_description)/meshes/hand_joint_side_plate_v4_1.stl" scale="0.001 0.001 0.001"/>
     </geometry>
   </collision>
@@ -493,5 +493,5 @@
     <origin xyz="-0.264826 0.05557 -0.627062" rpy="0 0 0"/>
     <geometry>
-      <mesh filename="file://$(find arm_description)/meshes/tool_joint_bearing_holders_v4_1.stl" scale="0.001 0.001 0.001"/>
+      <mesh filename="file://$(find rebel_arm_description)/meshes/tool_joint_bearing_holders_v4_1.stl" scale="0.001 0.001 0.001"/>
     </geometry>
     <material name="silver"/>
@@ -500,5 +500,5 @@
     <origin xyz="-0.264826 0.05557 -0.627062" rpy="0 0 0"/>
     <geometry>
-      <mesh filename="file://$(find arm_description)/meshes/tool_joint_bearing_holders_v4_1.stl" scale="0.001 0.001 0.001"/>
+      <mesh filename="file://$(find rebel_arm_description)/meshes/tool_joint_bearing_holders_v4_1.stl" scale="0.001 0.001 0.001"/>
     </geometry>
   </collision>
@@ -513,5 +513,5 @@
     <origin xyz="-0.264812 0.02757 -0.627062" rpy="0 0 0"/>
     <geometry>
-      <mesh filename="file://$(find arm_description)/meshes/tool_joint_motor_side_plate_right_v1_1.stl" scale="0.001 0.001 0.001"/>
+      <mesh filename="file://$(find rebel_arm_description)/meshes/tool_joint_motor_side_plate_right_v1_1.stl" scale="0.001 0.001 0.001"/>
     </geometry>
     <material name="silver"/>
@@ -520,5 +520,5 @@
     <origin xyz="-0.264812 0.02757 -0.627062" rpy="0 0 0"/>
     <geometry>
-      <mesh filename="file://$(find arm_description)/meshes/tool_joint_motor_side_plate_right_v1_1.stl" scale="0.001 0.001 0.001"/>
+      <mesh filename="file://$(find rebel_arm_description)/meshes/tool_joint_motor_side_plate_right_v1_1.stl" scale="0.001 0.001 0.001"/>
     </geometry>
   </collision>
@@ -533,5 +533,5 @@
     <origin xyz="-0.264808 0.01957 -0.627062" rpy="0 0 0"/>
     <geometry>
-      <mesh filename="file://$(find arm_description)/meshes/tool_joint_motor_side_plate_left_v6_1.stl" scale="0.001 0.001 0.001"/>
+      <mesh filename="file://$(find rebel_arm_description)/meshes/tool_joint_motor_side_plate_left_v6_1.stl" scale="0.001 0.001 0.001"/>
     </geometry>
     <material name="silver"/>
@@ -540,5 +540,5 @@
     <origin xyz="-0.264808 0.01957 -0.627062" rpy="0 0 0"/>
     <geometry>
-      <mesh filename="file://$(find arm_description)/meshes/tool_joint_motor_side_plate_left_v6_1.stl" scale="0.001 0.001 0.001"/>
+      <mesh filename="file://$(find rebel_arm_description)/meshes/tool_joint_motor_side_plate_left_v6_1.stl" scale="0.001 0.001 0.001"/>
     </geometry>
   </collision>
@@ -553,5 +553,5 @@
     <origin xyz="-0.284866 0.016559 -0.539562" rpy="0 0 0"/>
     <geometry>
-      <mesh filename="file://$(find arm_description)/meshes/tool_joint_motor_plate_v1_1.stl" scale="0.001 0.001 0.001"/>
+      <mesh filename="file://$(find rebel_arm_description)/meshes/tool_joint_motor_plate_v1_1.stl" scale="0.001 0.001 0.001"/>
     </geometry>
     <material name="silver"/>
@@ -560,5 +560,5 @@
     <origin xyz="-0.284866 0.016559 -0.539562" rpy="0 0 0"/>
     <geometry>
-      <mesh filename="file://$(find arm_description)/meshes/tool_joint_motor_plate_v1_1.stl" scale="0.001 0.001 0.001"/>
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